File: joystic-rj45.kicad_pcb (KiCad board)
At the start: 2 copper layers, 38 x 22 mm, 6 parts, among them CN1 1x5, CN2 1x8, CN3 1x2, CN4 1x2

Commit message: changed logo text, cleaned up silkscreen from overlapping pcb edge
Parts:
- added G***: LOGO, logos:gmlogo, B.Cu at (150.5, 116.0)
Other:
- board text removed: "good micros"
